File: KiCad/Workeeb.kicad_pcb (KiCad board)
At the start: 2 copper layers, 227 parts, among them J1 USB_C_Receptacle_USB2.0, U1 EFM32HG322F64G-C-QFP48

Commit message: Work towards getting decoupling caps and col routes in place
Parts:
- removed C_DEC2: 1uF, Capacitor_SMD:C_0402_1005Metric
- C_IOVDD0, C_IOVDD_0: moved to F.Cu
- moved J1 428.4 mm to (51.8, 28.6)
- moved SW_RESET1 80.0 mm to (407.2, 45.2)
- moved C_VREGO1 77.3 mm to (384.8, 53.8), turned to -90 degrees
- moved C_IOVDD_3 72.4 mm to (397.0, 45.2), turned to 90 degrees
- moved C_IOVDD_5 65.8 mm to (377.4, 45.0)
- moved C_AVDD_0 47.2 mm to (396.5, 51.1), turned to -90 degrees
- moved C_AVDD0 43.0 mm to (397.8, 51.1), turned to -90 degrees
- moved C_DEC1 4.04 mm to (386.6, 55.6)
- moved C_AVDD_1 2.55 mm to (395.5, 42.4), turned to -90 degrees
- moved C_DREG1 2.29 mm to (388.4, 53.1)
- moved C_DREG2 2.29 mm to (388.4, 54.1)
- moved C_IOVDD0 1.85 mm to (385.3, 36.8)
- moved C_IOVDD_0 1.61 mm to (385.3, 38.1)
- turned D103 to 180 degrees
Connections:
- D102 pad 1: unconnected-(D102-Pad1) -> GND
- D102 pad 2: unconnected-(D102-Pad2) -> NUMLK
- D103 pad 1: unconnected-(D103-Pad1) -> GND
- D103 pad 2: unconnected-(D103-Pad2) -> CAPS
Routing:
- net VDD: track 16.0 -> 55.1 mm, vias 6 -> 7
- net COL1: track 460.4 -> 487.4 mm
- net COL2: track 383.2 -> 409.5 mm
- net COL3: track 406.7 -> 432.3 mm
- net COL4: track 412.2 -> 437.5 mm
- net COL5: track 370.8 -> 395.0 mm
- net COL6: track 350.2 -> 371.7 mm
- net COL7: track 329.5 -> 350.4 mm
- net COL11: track 286.3 -> 303.3 mm
- net COL10: track 273.5 -> 290.5 mm
- net COL9: track 291.8 -> 308.7 mm
- net COL8: track 311.7 -> 328.6 mm
- net COL13: track 237.7 -> 254.4 mm
- net COL14: track 227.3 -> 244.0 mm
- net COL15: track 213.4 -> 230.1 mm
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Other:
- board outline added: 405.4 x 131.3 mm
