File: KiCad/Workeeb.kicad_pcb (KiCad board)
At the start: 2 copper layers, 405.4 x 131.3 mm, 226 parts, among them J1 USB_C_Receptacle_USB2.0, U1 EFM32HG322F64G-C-QFP48

Commit message: Connect up a bunch more stuff and set ground plane zone
Parts:
- C_RESET1: moved to F.Cu
- moved C_RESET1 78.4 mm to (392.4, 43.4), turned to 90 degrees
- moved R_RESET1 51.4 mm to (406.4, 42.0), turned to -90 degrees
- moved C_AVDD0 5.93 mm to (391.9, 50.0), turned to 180 degrees
- moved C_AVDD_0 5.00 mm to (391.9, 49.0), turned to 180 degrees
- moved C_IOVDD_3 4.85 mm to (393.4, 48.5), turned to -90 degrees
- moved C_AVDD_1 4.22 mm to (393.7, 46.2), turned to 0 degrees
- moved C_VREGO1 2.50 mm to (383.8, 51.6)
- moved C_DEC1 2.29 mm to (388.8, 55.2), turned to 0 degrees
- moved C_DREG1 0.48 mm to (388.8, 53.1)
- moved C_DREG2 0.48 mm to (388.8, 54.1)
Routing:
- net ROW6: track 360.3 -> 468.4 mm, vias 0 -> 2
- net ROW5: track 391.2 -> 483.1 mm, vias 0 -> 2
- net ROW4: track 346.9 -> 424.4 mm, vias 0 -> 2
- net ROW3: track 396.0 -> 455.3 mm, vias 0 -> 2
- net ROW2: track 381.0 -> 427.0 mm, vias 0 -> 2
- net ROW1: track 313.9 -> 359.0 mm
- net COL20: track 66.3 -> 100.3 mm
- net NUMLK: track 0.00 -> 32.6 mm, vias 0 -> 1
- net RESET: track 0.00 -> 26.5 mm, vias 0 -> 1
- net CAPS: track 0.00 -> 25.1 mm, vias 0 -> 1
- net COL18: track 80.0 -> 97.3 mm
- net COL19: track 75.8 -> 90.7 mm
- net VBUS: track 0.00 -> 6.44 mm
- net Net-(C_DEC1-Pad1): track 0.00 -> 6.33 mm
- net VDD: track 55.1 -> 58.2 mm
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- added copper zone on B.Cu, net GND
- added copper zone on F.Cu, net GND
