File: KiCad/Workeeb.kicad_sch (KiCad schematic)
At the start: 228 parts, among them J1 USB_C_Receptacle_USB2.0, U1 EFM32HG322F64G-C-QFP48

Commit message: finish up DRC warns/errs
Parts:
- added R_BADGE1: 500, Resistor_SMD:R_0805_2012Metric, symbol Device:R
- renumbered R_CAPS to R_CAPS1, R_NUMLK to R_NUMLK1
Connections:
- net BADGE: now also R_BADGE1.1; no longer D101.2 (DIN)
- new net: D101.2 (DIN), R_BADGE1.2
Changed lines of the file:
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@@
     )
   )
-  (global_label "BADGE" (shape input) (at 406.4 113.03 180) (fields_autoplaced)
+  (global_label "BADGE" (shape input) (at 398.78 113.03 180) (fields_autoplaced)
     (effects (font (size 1.27 1.27)) (justify right))
-    (property "Intersheet References" "${INTERSHEET_REFS}" (id 0) (at 398.0282 113.1094 0)
+    (property "Intersheet References" "${INTERSHEET_REFS}" (id 0) (at 390.4082 113.1094 0)
       (effects (font (size 1.27 1.27)) (justify right) hide)
     )
@@
   (symbol (lib_id "Device:R") (at 443.23 120.65 90) (unit 1)
     (in_bom yes) (on_board yes)
-    (property "Reference" "R_CAPS" (id 0) (at 443.23 118.11 90))
+    (property "Reference" "R_CAPS1" (id 0) (at 443.23 118.11 90))
     (property "Value" "10" (id 1) (at 443.23 120.65 90))
     (property "Footprint" "Resistor_SMD:R_0805_2012Metric" (id 2) (at 443.23 122.428 90)
@@
   (symbol (lib_id "Device:R") (at 443.23 111.76 90) (unit 1)
     (in_bom yes) (on_board yes)
-    (property "Reference" "R_NUMLK" (id 0) (at 443.23 109.22 90))
+    (property "Reference" "R_NUMLK1" (id 0) (at 443.23 109.22 90))
     (property "Value" "10" (id 1) (at 443.23 111.76 90))
     (property "Footprint" "Resistor_SMD:R_0805_2012Metric" (id 2) (at 443.23 113.538 90)
@@
     (pin "2")
   )
+  (symbol (lib_id "Device:R") (at 402.59 113.03 90) (unit 1)
+    (in_bom yes) (on_board yes)
+    (property "Reference" "R_BADGE1" (id 0) (at 402.59 110.49 90))
+    (property "Value" "500" (id 1) (at 402.59 113.03 90))
+    (property "Footprint" "Resistor_SMD:R_0805_2012Metric" (id 2) (at 402.59 114.808 90)
+      (effects (font (size 1.27 1.27)) hide)
+    )
+    (property "Datasheet" "~" (id 3) (at 402.59 113.03 0)
+      (effects (font (size 1.27 1.27)) hide)
+    )
+    (pin "1")
+    (pin "2")
+  )
   (symbol (lib_id "power:VDD") (at 364.49 62.23 270) (unit 1)
     (in_bom yes) (on_board yes) (fields_autoplaced)
@@
       (reference "MX100") (unit 1) (value "numEnter") (footprint "MX_Only:MXOnly-2U-VerticalStabilizers-NoLED")
     )
+    (path "/b780a946-6c5d-4028-a561-8dbe67d7e077"
+      (reference "R_BADGE1") (unit 1) (value "500") (footprint "Resistor_SMD:R_0805_2012Metric")
+    )
     (path "/0fff7ce4-a8e7-44cd-ae3c-b49dae575d0f"
-      (reference "R_CAPS") (unit 1) (value "10") (footprint "Resistor_SMD:R_0805_2012Metric")
+      (reference "R_CAPS1") (unit 1) (value "10") (footprint "Resistor_SMD:R_0805_2012Metric")
     )
     (path "/95da3e95-4c59-46e8-9744-59a7567d7f21"
@@
     )
     (path "/a840eb2a-84fd-40d8-ab3f-ff2711691f52"
-      (reference "R_NUMLK") (unit 1) (value "10") (footprint "Resistor_SMD:R_0805_2012Metric")
+      (reference "R_NUMLK1") (unit 1) (value "10") (footprint "Resistor_SMD:R_0805_2012Metric")
     )
     (path "/ec0c6572-a860-4bd5-b379-196b962533e8"
